File: DYI-LORA-PCB/DYI-LORA-PCB.kicad_pcb (KiCad board)
At the start: 2 copper layers, 67 parts, among them J1 Conn_01x06_Pin, J2 Conn_Coaxial, J3 Conn_01x05_Pin, J4 VIB-MOTOR Connector, J5 Conn_01x04_Pin, J7 USB_B_Micro, J8 Conn_01x02_Pin, Q1 AO3400A, Q2 FS8205A, Q3 AO3401A, Q4 MMBT2222A, SW1 SW_PushReset, SW2 SW_PushBoot, SW3 MTS-102, U1 ESP32-S3-WROOM-1, U10 DW01A, U11 AP2112K-3.3, U2 RFM9X, U3 QMC5883P, U4 PCF85063ATL, U8 TP4056-42-ESOP8, U9 USBLC6-2SC6, Y1 Crystal

Commit message: journal 7
Parts:
- removed R7, R8: 4.7k, Resistor_SMD:R_0805_2012Metric_Pad1.20x1.40mm_HandSolder
- added R22: 10kiloOhms, Resistor_SMD:R_1206_3216Metric_Pad1.30x1.75mm_HandSolder, F.Cu at (51.8, 84.5)
- added REF**: MountingHole_3.2mm_M3, MountingHole:MountingHole_3.2mm_M3, F.Cu at (24.5, 49.0)
- added REF**: MountingHole_3.2mm_M3, MountingHole:MountingHole_3.2mm_M3, F.Cu at (24.5, 124.0)
- added REF**: MountingHole_3.2mm_M3, MountingHole:MountingHole_3.2mm_M3, F.Cu at (125.0, 49.0)
- added REF**: MountingHole_3.2mm_M3, MountingHole:MountingHole_3.2mm_M3, F.Cu at (124.5, 124.0)
- D6, Q4, R13, R14, R16, R17: moved to B.Cu
- moved R13 119.1 mm to (66.5, 86.0), turned to -90 degrees
- moved D6 116.8 mm to (65.5, 81.0), turned to -90 degrees
- moved R14 115.5 mm to (70.5, 87.5), turned to 0 degrees
- moved Q4 112.4 mm to (70.5, 83.5), turned to 90 degrees
- moved BZ1 105.9 mm to (70.5, 74.0), turned to -90 degrees
- moved C9 66.6 mm to (47.5, 86.0)
- moved C3 50.0 mm to (38.0, 80.5)
- moved R16 48.3 mm to (37.0, 58.0)
- moved R17 43.1 mm to (41.0, 55.5), turned to -90 degrees
- moved J3 36.4 mm to (26.0, 86.6)
- moved SW3 33.1 mm to (89.2, 115.2)
- moved C7 11.2 mm to (47.5, 84.0)
- moved C4 7.81 mm to (108.5, 63.5)
- moved C6 7.81 mm to (108.5, 61.0)
- moved R3 7.81 mm to (111.0, 86.0)
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Connections:
- J1 pad 5: unconnected-(J1-Pin_5-Pad5) -> Net-(J1-Pin_5)
- R16 pad 2: unconnected-(R16-Pad2) -> SDA-KB
- U1 pad 8: TX-GPS -> RX-GPS
- U1 pad 9: RX-GPS -> TX-GPS
- U2 pad 1: GND -> PROT-GND
- U2 pad 10: GND -> PROT-GND
- U2 pad 8: GND -> PROT-GND
Routing:
- net +3.3V: track 85.3 -> 312.1 mm, vias 5 -> 14
- net PROT-GND: track 158.1 -> 246.7 mm, vias 16 -> 20
- net RESET: track 0.00 -> 68.4 mm, vias 0 -> 1
- net NSS-RFM: track 0.00 -> 67.9 mm, vias 0 -> 1
- net SCK-RFM: track 0.00 -> 62.7 mm, vias 0 -> 3
- net DIO1-RFM: track 0.00 -> 61.5 mm, vias 0 -> 1
- net MOSI-RFM: track 0.00 -> 59.1 mm, vias 0 -> 1
- net DIO0-RFM: track 0.00 -> 55.3 mm, vias 0 -> 1
- net MISO-RFM: track 0.00 -> 55.1 mm, vias 0 -> 1
- net GND: track 53.8 -> 0.00 mm
- net VIB-MOTOR-CTRL: track 0.00 -> 50.8 mm, vias 0 -> 4
- net ADC-PIN: track 4.78 -> 45.3 mm, vias 0 -> 2
- net SCL-KB: track 1.16 -> 39.7 mm, vias 1 -> 5
- net D+: track 6.76 -> 42.8 mm, vias 0 -> 2
- net D-: track 4.41 -> 40.3 mm, vias 2 -> 3
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Other:
- board outline added: 110.4 x 85 mm
- board text added: "Battery"
- board text added: "GPS"
