File: DYI-LORA-PCB/DYI-LORA-PCB.kicad_sch (KiCad schematic)
At the start: 19 parts, among them J1 USB_B_Micro, J2 Conn_Coaxial, J3 Conn_01x08_Pin, SW1 SW_PushReset, SW2 SW_PushBoot, U1 ESP32-S3-WROOM-1, U2 RFM9X, U3 AMS1117-3.3, U4 USBLC6-2SC6

Commit message: journal 3
Parts:
- removed C1: 10microFarad, Capacitor_SMD:C_0805_2012Metric_Pad1.18x1.45mm_HandSolder, symbol Device:C_Small
- removed C2: 22microFarad, Capacitor_SMD:C_1206_3216Metric_Pad1.33x1.80mm_HandSolder, symbol Device:C_Small
- removed J1: USB_B_Micro, symbol Connector:USB_B_Micro
- removed J3: Conn_01x08_Pin, Connector_PinHeader_2.54mm:PinHeader_1x08_P2.54mm_Vertical, symbol Connector:Conn_01x08_Pin
- removed U3: AMS1117-3.3, Package_TO_SOT_SMD:SOT-223-3_TabPin2, symbol Regulator_Linear:AMS1117-3.3
- removed U4: USBLC6-2SC6, Package_TO_SOT_SMD:SOT-23-6, symbol Power_Protection:USBLC6-2SC6
- added BZ1: Buzzer, Buzzer_Beeper:MagneticBuzzer_PUI_AT-0927-TT-6-R, symbol Device:Buzzer
- added C10: 4.7microF, Capacitor_SMD:C_0805_2012Metric_Pad1.18x1.45mm_HandSolder, symbol Device:C_Small
- added C11, C12, C13: 10microFarad, Capacitor_SMD:C_0805_2012Metric_Pad1.18x1.45mm_HandSolder, symbol Device:C_Small
- added C14: 22microFarad, Capacitor_SMD:C_1206_3216Metric_Pad1.33x1.80mm_HandSolder, symbol Device:C_Small
- added C15: 0.22microF, Capacitor_SMD:C_0805_2012Metri, symbol Device:C_Small
- added C16, C17, C9: 100nanoFarad, Capacitor_SMD:C_0603_1608Metric_Pad1.08x0.95mm_HandSolder, symbol Device:C_Small
- added C7: 10microF, Capacitor_SMD:C_0805_2012Metric_Pad1.18x1.45mm_HandSolder, symbol Device:C_Small
- added C8: C-IN-10microF, Capacitor_SMD:C_0805_2012Metric_Pad1.18x1.45mm_HandSolder, symbol Device:C_Small
- added D1: 1N5819, Diode_SMD:D_SOD-123, symbol Device:D
- added D2: D_Schottky, symbol Device:D_Schottky
- added D4: LED RED, LED_SMD:LED_0805_2012Metric_Pad1.15x1.40mm_HandSolder, symbol Device:LED
- added D5: LED BLUE, LED_SMD:LED_0805_2012Metric_Pad1.15x1.40mm_HandSolder, symbol Device:LED
- added D6: 1N4148W, Diode_SMD:D_SOD-123, symbol Diode:1N4148W
- added F2: Fuse 1.1A hold, symbol Device:Fuse
- added J1: Conn_01x06_Pin, Connector_JST:JST_SH_SM06B-SRSS-TB_1x06-1MP_P1.00mm_Horizontal, symbol Connector:Conn_01x06_Pin
- added J3: Conn_01x05_Pin, Connector_PinHeader_2.54mm:PinHeader_1x05_P2.54mm_Vertical, symbol Connector:Conn_01x05_Pin
- added J4: VIB-MOTOR Connector, Connector_PinHeader_2.54mm:PinHeader_1x02_P2.54mm_Vertical, symbol Connector:Conn_01x02_Pin
- added J5: Conn_01x04_Pin, Connector_JST:JST_SH_SM04B-SRSS-TB_1x04-1MP_P1.00mm_Horizontal, symbol Connector:Conn_01x04_Pin
- added J7: USB_B_Micro, Connector_USB:USB_Micro-B_Molex_47346-0001, symbol Connector:USB_B_Micro
- added J8: Conn_01x02_Pin, Connector_JST:JST_PH_S2B-PH-K_1x02_P2.00mm_Horizontal, symbol Connector:Conn_01x02_Pin
- added Q1: AO3400A, Package_TO_SOT_SMD:SOT-23_Handsoldering, symbol Transistor_FET:AO3400A
- added Q2: FS8205A, Package_SO:TSSOP-8_4.4x3mm_P0.65mm, symbol FS8205A:FS8205A
- added Q3: AO3401A, Package_TO_SOT_SMD:SOT-23_Handsoldering, symbol Transistor_FET:AO3401A
- added Q4: MMBT2222A, Package_TO_SOT_SMD:SOT-23_Handsoldering, symbol Transistor_BJT:MMBT2222A
- added R10, R11: 1k ohms, Resistor_SMD:R_1206_3216Metric_Pad1.30x1.75mm_HandSolder, symbol Device:R
- added R12: 1.2kΩ (≈1A) or 2.4kΩ (≈500mA), Resistor_SMD:R_1206_3216Metric_Pad1.30x1.75mm_HandSolder, symbol Device:R
- added R13, R14: 1k, Resistor_SMD:R_0805_2012Metric_Pad1.20x1.40mm_HandSolder, symbol Device:R
- added R5: 100 ohms, Resistor_SMD:R_1206_3216Metric_Pad1.30x1.75mm_HandSolder, symbol Device:R
- added R6: 100k ohms, Resistor_SMD:R_1206_3216Metric_Pad1.30x1.75mm_HandSolder, symbol Device:R
- added R7, R8: 4.7k, Resistor_SMD:R_0805_2012Metric_Pad1.20x1.40mm_HandSolder, symbol Device:R
- added R9: 100k, Resistor_SMD:R_0805_2012Metric_Pad1.20x1.40mm_HandSolder, symbol Device:R
- added SW3: MTS-102, symbol Switch:SW_SPDT
- added U10: DW01A, Package_TO_SOT_SMD:SOT-23-6, symbol Battery_Management:DW01A
- added U11: AP2112K-3.3, Package_TO_SOT_SMD:SOT-23-5_HandSoldering, symbol Regulator_Linear:AP2112K-3.3
- added U3: QMC5883P, Package_LGA:LGA-16_3x3mm_P0.5mm, symbol qmc5883p:QMC5883P
- added U4: PCF85063ATL, Package_DFN_QFN:DFN-10-1EP_2.6x2.6mm_P0.5mm_EP1.3x2.2mm, symbol Timer_RTC:PCF85063ATL
- added U8: TP4056-42-ESOP8, Package_SO:SOIC-8-1EP_3.9x4.9mm_P1.27mm_EP2.41x3.3mm_ThermalVias, symbol Battery_Management:TP4056-42-ESOP8
- added U9: USBLC6-2SC6, Package_TO_SOT_SMD:SOT-23-6, symbol Power_Protection:USBLC6-2SC6
Connections:
- net +3.3V: now also BZ1.1 (+), C14.1, C16.1, D1.1 (K), D6.1 (K), J3.1 (Pin_1), J4.1 (Pin_1), J5.2 (Pin_2), R7.2, R8.2, U11.5 (VOUT), U3.13 (NC), U3.4 (NC)
- net CS-DISPLAY: now also J3.5 (Pin_5)
- net D+: now also J7.3 (D+), U9.3 (I/O2), U9.5 (VBUS)
- net D-: now also J7.2 (D-), U9.1 (I/O1), U9.6 (I/O1)
- net GND: no longer C3.1, C4.2, C6.2, U1.1 (GND), U1.40 (GND), U1.41 (GND)
- net PROT-GND: now reaches SW2.1
- net PROT-GND: now also C3.1, C4.2, C6.2, SW1.1, U1.1 (GND), U1.40 (GND), U1.41 (GND), C10.2, C13.1, C14.2, C7.2, C9.2, J1.2 (Pin_2), J3.2 (Pin_2), J5.1 (Pin_1), J7.5 (GND), J7.SH (Shield), Q1.2 (S), Q2.6, Q2.7, Q4.2 (E), R14.1, R6.2, U10.6 (GND), U11.2 (GND), U3.11 (GND), U3.9 (GND), U9.2 (GND)
- net BUZZER-GPIO: now reaches U1.11 (GPIO18/U1RXD/ADC2_CH7/CLK_OUT3)
- net BUZZER-GPIO: now also R13.1
- net SDA-QMC: now reaches U1.23 (GPIO21)
- net SDA-QMC: now also R7.1, U3.16 (SDA)
- net SCK-QMC: now reaches U1.24 (GPIO47/SPICLK_P/SUBSPICLK_P_DIFF)
- net SCK-QMC: now also R8.1, U3.1 (SCK)
- net SCL-KB: now reaches U1.38 (GPIO2/TOUCH2/ADC1_CH1)
- net SCL-KB: now also J5.4 (Pin_4)
- net SDA-KB: now reaches U1.39 (GPIO1/TOUCH1/ADC1_CH0)
- net SDA-KB: now also J5.3 (Pin_3)
- net VIB-MOTOR-CTRL: now reaches U1.7 (GPIO7/TOUCH7/ADC1_CH6)
- net VIB-MOTOR-CTRL: now also R5.1
- net TX-GPS: now reaches U1.8 (GPIO15/U0RTS/ADC2_CH4/XTAL_32K_P)
- net TX-GPS: now also J1.4 (Pin_4)
- net RX-GPS: now reaches U1.9 (GPIO16/U0CTS/ADC2_CH5/XTAL_32K_N)
- net RX-GPS: now also J1.3 (Pin_3)
- net DC-DISPLAY: no longer names the net of U1.31 (GPIO38/FSPIWP/SUBSPIWP)
- net RES-DISPLAY: no longer names the net of U1.32 (MTCK/GPIO39/CLK_OUT3/SUBSPICS1)
- net SCL-DISPLAY renamed MOSI-DISPLAY
- net MOSI-DISPLAY: now also J3.4 (Pin_4)
- net SDA-DISPLAY renamed SCK-DISPLAY
- net SCK-DISPLAY: now also J3.3 (Pin_3)
- new net: D4.1 (K), U8.7 (~{CHRG})
- new net: D4.2 (A), R10.2
- new net: D5.2 (A), R11.2
- new net: R12.2, U8.2 (PROG)
- new net: D5.1 (K), U8.6 (~{STDBY})
- new net: C10.1, U3.10 (C1)
- new net: C15.2, U3.12 (NC)
- new net: C15.1, U3.8 (NC)
- new net: Q4.1 (B), R13.2, R14.2
- new net: BZ1.2 (-), D6.2 (A), Q4.3 (C)
- new net: Q3.1 (G), R9.2
- new net: Q1.1 (G), R5.2, R6.1
- new net: F2.1, J8.1 (Pin_1)
- new net: D1.2 (A), J4.2 (Pin_2), Q1.3 (D)
- new net BATT+: C12.2, C7.1, C9.1, F2.2, J1.1 (Pin_1), Q3.2 (S), U10.5 (VCC), U8.5 (BAT)
- new net BATT-: C11.1, C12.1, J8.2 (Pin_2), Q2.2, Q2.3, R12.1, U8.3 (GND), U8.9 (EPAD)
- new net CS-DW01A: Q2.1, Q2.8, U10.2 (CS)
- new net OC-DW01A: Q2.5, U10.3 (OC)
- new net OD-DW01A: Q2.4, U10.1 (OD)
- new net SYS_PWR: C13.2, D2.1 (K), Q3.3 (D), U11.1 (VIN), U11.3 (EN)
- new net VBUS: C11.2, D2.2 (A), J7.1 (VBUS), R10.1, R11.1, R9.1, U8.4 (V_{CC}), U8.8 (CE), U9.4 (I/O2)
- no-connect marks 0 -> 2
Other:
- note added: "APK2112K-3.3"
- note added: "BAT"
- note added: "Buzzer"
- note added: "DW01A"
- note added: "FS8205A"
- note added: "GPS Vollgo VG7669T160N0MA"
- note added: "Laskakit Mem LCD DIsplay"
- note added: "M5 Stack CardKB"
- note added: "MCU"
- note added: "MICRO-USB + ESD"
- note added: "Power"
- note added: "QST QMC5883P"
- note added: "RTC"
- note added: "TP4056"
- note added: "Vibration Motor"
- moved on the sheet: C3, C5, R1, R2, SW1, SW2, U1

Commit message: journal 4
Parts:
- added C18: 100nanoFarad, Capacitor_SMD:C_0603_1608Metric_Pad1.08x0.95mm_HandSolder, symbol Device:C_Small
- added R15, R16, R17, R18, R19: 10kiloOhms, Resistor_SMD:R_1206_3216Metric_Pad1.30x1.75mm_HandSolder, symbol Device:R
- added Y1: Crystal, Crystal:Crystal_SMD_3215-2Pin_3.2x1.5mm, symbol Device:Crystal
Connections:
- net +3.3V: now also C7.1, C9.1, J1.1 (Pin_1), R16.1, R17.1
- net BATT+: now also R18.1; no longer C7.1, C9.1, J1.1 (Pin_1)
- net BATT-: now also R19.2
- net PROT-GND: now also U4.5 (VSS), C18.1
- net SCL-KB: now also U4.7 (SCL), R17.2
- net SDA-KB: now also U4.6 (SDA)
- net TEMP: now reaches U8.1 (TEMP)
- net TEMP: now also R18.2, R19.1
- net at U4.1 (OSCI): now also Y1.1
- net at U4.10 (VDD): now also C18.2, R15.1
- net at U4.2 (OSCO): now also Y1.2
- net INT-RTC: now reaches U4.4 (~{INT})
- net INT-RTC: now also U1.31 (GPIO38/FSPIWP/SUBSPIWP), R15.2
Other:
- moved on the sheet: SW3, U4

Commit message: journal 5 and 6
Parts:
- added C19: 100nanoFarad, Capacitor_SMD:C_0603_1608Metric_Pad1.08x0.95mm_HandSolder, symbol Device:C_Small
- added R20, R21: 100kiloOhms, Resistor_SMD:R_1206_3216Metric_Pad1.30x1.75mm_HandSolder, symbol Device:R
- D2: value D_Schottky -> 1N5819W; footprint (none) -> Diode_SMD:D_SOD-123
- F2: footprint (none) -> Fuse:Fuse_1206_3216Metric_Pad1.42x1.75mm_HandSolder
- SW3: footprint (none) -> Button_Switch_THT:SW_CW_GPTS203211B
Connections:
- net +3.3V: now also SW3.1 (A), U2.13 (VDD); no longer C14.1, U11.5 (VOUT), U2.12 (VDD)
- net BATT+: now also R20.1
- net BATT-: now also C19.2, R21.2
- net DIO0-RFM: now also U2.14 (DIO0); no longer U2.11 (DIO0)
- net DIO1-RFM: now also U2.15 (DIO1); no longer U2.10 (DIO1)
- net GND: now also U2.10 (GND); no longer C5.2, U2.15 (GND)
- net NSS-RFM: now also R3.2
- net PROT-GND: now also C16.2, C5.2
- net 3.3V-RTC: now reaches C18.2, R15.1, U4.10 (VDD)
- net 3.3V-RTC: now also C14.1, SW3.2 (B), U11.5 (VOUT)
- net ADC-PIN: now reaches U1.15 (GPIO3/TOUCH3/ADC1_CH2)
- net ADC-PIN: now also C19.1, R20.2, R21.1
- net at J2.1 (In): now also U2.9 (ANT); no longer U2.16 (ANT)
Other:
- moved on the sheet: C11, C17, C8, SW3

Commit message: journal 7
Parts:
- removed R7, R8: 4.7k, Resistor_SMD:R_0805_2012Metric_Pad1.20x1.40mm_HandSolder, symbol Device:R
- added R22: 10kiloOhms, Resistor_SMD:R_1206_3216Metric_Pad1.30x1.75mm_HandSolder, symbol Device:R
Connections:
- net +3.3V: now also R22.1
- net GND: no longer U2.1 (GND), U2.10 (GND), U2.8 (GND)
- net PROT-GND: now also U2.1 (GND), U2.10 (GND), U2.8 (GND)
- net RX-GPS: now also U1.8 (GPIO15/U0RTS/ADC2_CH4/XTAL_32K_P); no longer U1.9 (GPIO16/U0CTS/ADC2_CH5/XTAL_32K_N)
- net SDA-KB: now also R16.2
- net TX-GPS: now also U1.9 (GPIO16/U0CTS/ADC2_CH5/XTAL_32K_N); no longer U1.8 (GPIO15/U0RTS/ADC2_CH4/XTAL_32K_P)
- net at J1.5 (Pin_5): now also R22.2
- no-connect marks 2 -> 1
Other:
- moved on the sheet: R16
